File: board/main.brd (EAGLE design)
At the start: 37.8 x 39.4 mm, 11 parts, among them Q1 12MHz, U1 ATMEGA328P_TQFP

Commit message: Finished routing
Signed-off-by: Garrett Greenwood <garrettagreenwood@gmail.com>
Parts:
- added C3, C4: .1uF, resistor:C0603
- moved MISC 8.87 mm to (10.4, 26.4)
- moved C1 8.68 mm to (8.80, 16.8), turned to 270 degrees
- moved DIGITAL 8.57 mm to (22.4, 26.4)
- moved Q1 8.25 mm to (7.60, 10.8)
- moved U$1 6.53 mm to (30.4, 12.0)
- moved U1 6.09 mm to (19.2, 14.4)
- moved C2 5.74 mm to (5.60, 16.8), turned to 270 degrees
- moved ANALOG 4.89 mm to (28.8, 4.00)
- moved GCN 4.75 mm to (9.60, 4.00)
- moved DPAD 4.66 mm to (18.4, 4.00)
- moved ISP1 4.02 mm to (34.4, 21.2), turned to 90 degrees
Connections:
- net 3V3: now also C3.1
- net 5V: now also C4.1
- net GND: now also C3.2, C4.2, MISC.1, U1.21
Routing:
- net 3V3: track 0.00 -> 74.6 mm, vias 0 -> 3
- net 5V: track 0.00 -> 43.6 mm
- net GND: track 0.00 -> 40.7 mm, vias 0 -> 1
- net SCK: track 0.00 -> 28.2 mm, vias 0 -> 1
- net MOSI: track 0.00 -> 28.2 mm
- net AVR_RESET: track 0.00 -> 25.7 mm, vias 0 -> 1
- net N$2: track 0.00 -> 24.9 mm
- net N$4: track 0.00 -> 23.0 mm, vias 0 -> 1
- net SS: track 0.00 -> 19.7 mm
- net N$19: track 0.00 -> 15.0 mm
- net N$5: track 0.00 -> 14.4 mm
- net N$18: track 0.00 -> 14.0 mm
- net N$20: track 0.00 -> 13.0 mm
- net N$6: track 0.00 -> 12.3 mm
- net N$7: track 0.00 -> 11.1 mm
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- added copper zone on layer 1, net GND
- added copper zone on layer 16, net GND
Other:
- board size 37.8 x 39.4 mm -> 40 x 30.4 mm
- board text added: "3V3"
- board text added: "5V"
- board text added: "DO"
- board text added: "GND"
- board text added: "LE"
- board text added: "RI"
- board text added: "SIG"
- board text added: "UP"
- board text added: "X1"
- board text added: "X2"
- board text added: "Y1"
- board text added: "Y2"
- board text added: "Z1"
- board text added: "Z2"

Commit message: Completed v0.1 of PCB
Signed-off-by: Garrett Greenwood <garrettagreenwood@gmail.com>
Connections:
- net N$10 renamed Z1
- net N$11 renamed X2
- net N$12 renamed Y2
- net N$13 renamed Z3
- net N$14 renamed D_LEFT
- net N$15 renamed D_DOWN
- net N$16 renamed D_RIGHT
- net N$17 renamed D_UP
- net N$18 renamed GCN_SIG
- net N$19 renamed XBOX_RESET
- net N$20 renamed USB_D-
- net N$21 renamed VIEW
- net N$22 renamed XBOX
- net N$23 renamed MENU
- net N$24 renamed R
- net N$25 renamed L
- net N$3 renamed X1
- net N$5 renamed A
- net N$6 renamed B
- net N$7 renamed X
- net N$8 renamed Y
- net N$9 renamed Y1
Other:
- board text added: "A"
- board text added: "B"
- board text added: "D-"
- board text added: "GARRETT GREENWOOD GAMECUBE->XBOX ONE ADAPTER V0.1"
- board text added: "L"
- board text added: "MENU"
- board text added: "R"
- board text added: "RST"
- board text added: "VIEW"
- board text added: "X"
- board text added: "XBOX"
- board text added: "Y"

Commit message: Ready to order v0.2 boards
Signed-off-by: Garrett Greenwood <garrettagreenwood@gmail.com>
Parts:
- removed DIGITAL: 53047-09, con-molex:53047-09
- removed Q1: 12MHz, crystal:CTS406
- added Q2: 12MHz, crystal:HC49/S
- added R1: 10k, resistor:R0603
- added U$6: 1X9, headers(2mm):1X9
- ANALOG: value 53047-06 -> 1X6; device con-molex:53047-06 -> headers(2mm):1X6
- DPAD: value 53047-05 -> 1X4; device con-molex:53047-05 -> headers(2mm):1X4
- GCN: value 53047-04 -> 1X4; device con-molex:53047-04 -> headers(2mm):1X4
- MISC: value 53047-05 -> 1X5; device con-molex:53047-05 -> headers(2mm):1X5
- moved ANALOG 1.92 mm to (30.0, 2.50), turned to 0 degrees
- moved MISC 1.71 mm to (11.0, 28.0)
- moved DPAD 1.62 mm to (19.0, 2.50), turned to 0 degrees
- moved GCN 1.55 mm to (10.0, 2.50)
- renumbered U$1 to DAC
Connections:
- net XBOX_RESET renamed MISC-RST
- removed net D_DOWN: DPAD.4, U1.12
- removed net D_LEFT: DPAD.5, U1.13
- removed net D_RIGHT: DPAD.3, U1.11
- removed net D_UP: DPAD.2, U1.10
- removed net USB_D-: MISC.2, U1.1
- new net DPAD-D: DPAD.3, U1.12
- new net DPAD-L: DPAD.4, U1.13
- new net DPAD-R: DPAD.2, U1.11
- new net DPAD-U: DPAD.1, U1.10
- new net MISC-D-: MISC.4, U1.1
- net 3V3: now also MISC.2, R1.2; no longer MISC.4
- net 5V: now also MISC.1; no longer MISC.5
- net A: now also U$6.9; no longer DIGITAL.1
- net B: now also U$6.8; no longer DIGITAL.2
- net GCN_SIG: now also R1.1
- net GND: now also MISC.5; no longer DPAD.1, MISC.1
- net L: now also U$6.5; no longer DIGITAL.5
- net MENU: now also U$6.3; no longer DIGITAL.7
- net N$1: now also Q2.2; no longer Q1.3
- net N$2: now also Q2.1; no longer Q1.1
- net R: now also U$6.4; no longer DIGITAL.6
- net VIEW: now also U$6.1; no longer DIGITAL.9
- net X: now also U$6.7; no longer DIGITAL.3
- net XBOX: now also U$6.2; no longer DIGITAL.8
- net Y: now also U$6.6; no longer DIGITAL.4
Routing:
- net USB_D-: track 13.0 -> 0.00 mm
- net MISC-D-: track 0.00 -> 12.7 mm
- net DPAD-L: track 0.00 -> 10.0 mm
- net 5V: track 43.6 -> 34.5 mm
- net DPAD-U: track 0.00 -> 8.81 mm
- net DPAD-D: track 0.00 -> 8.81 mm
- net A: track 14.4 -> 23.1 mm
- net B: track 12.3 -> 20.3 mm
- net D_LEFT: track 7.86 -> 0.00 mm
- net DPAD-R: track 0.00 -> 7.61 mm
- net D_DOWN: track 7.41 -> 0.00 mm
- net X: track 11.1 -> 18.3 mm
- net D_RIGHT: track 6.96 -> 0.00 mm
- net D_UP: track 6.61 -> 0.00 mm
- net Y: track 10.6 -> 17.1 mm
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Other:
- board size 40 x 30.4 mm -> 42 x 30.4 mm
- board text added: "GARRETT GREENWOOD GAMECUBE->XBOX ONE ADAPTER V0.2"
- board text removed: "GARRETT GREENWOOD GAMECUBE->XBOX ONE ADAPTER V0.1"
