File: board/main.sch (EAGLE design)
At the start: 11 parts, among them Q1 12MHz, U1 ATMEGA328P_TQFP

Commit message: Finished routing
Signed-off-by: Garrett Greenwood <garrettagreenwood@gmail.com>
Parts:
- added C3, C4: .1uF, resistor:C-EUC0603
Connections:
- net 3V3: now also C3.1
- net 5V: now also C4.1
- net GND: now also C3.2, C4.2, MISC-1.S, U1.AGND
Changed lines of the file:
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@@
 <part name="DIGITAL" library="con-molex" deviceset="53?-09" device="047"/>
 <part name="GND5" library="supply1" deviceset="GND" device=""/>
+<part name="C3" library="resistor" deviceset="C-EU" device="C0603" value=".1uF"/>
+<part name="C4" library="resistor" deviceset="C-EU" device="C0603" value=".1uF"/>
 </parts>
 <sheets>
@@
 <instance part="ISP1" gate="G$1" x="137.16" y="30.48"/>
 <instance part="U1" gate="U$1" x="81.28" y="58.42"/>
-<instance part="GND2" gate="1" x="53.34" y="25.4"/>
+<instance part="GND2" gate="1" x="50.8" y="20.32"/>
 <instance part="GND3" gate="1" x="154.94" y="22.86"/>
 <instance part="GND4" gate="1" x="109.22" y="12.7" rot="R90"/>
@@
 <instance part="DIGITAL" gate="-9" x="109.22" y="60.96"/>
 <instance part="GND5" gate="1" x="104.14" y="111.76" rot="R270"/>
+<instance part="C3" gate="G$1" x="43.18" y="35.56" rot="R90"/>
+<instance part="C4" gate="G$1" x="43.18" y="27.94" rot="R90"/>
 </instances>
 <busses>
@@
 <wire x1="30.48" y1="60.96" x2="27.94" y2="60.96" width="0.1524" layer="91"/>
 <pinref part="GND1" gate="1" pin="GND"/>
+<junction x="30.48" y="60.96"/>
 </segment>
 <segment>
 <pinref part="U1" gate="U$1" pin="GND@3"/>
-<wire x1="55.88" y1="35.56" x2="53.34" y2="35.56" width="0.1524" layer="91"/>
-<wire x1="53.34" y1="35.56" x2="53.34" y2="33.02" width="0.1524" layer="91"/>
+<wire x1="55.88" y1="35.56" x2="50.8" y2="35.56" width="0.1524" layer="91"/>
+<wire x1="50.8" y1="35.56" x2="50.8" y2="33.02" width="0.1524" layer="91"/>
 <pinref part="U1" gate="U$1" pin="GND@5"/>
-<wire x1="55.88" y1="33.02" x2="53.34" y2="33.02" width="0.1524" layer="91"/>
-<wire x1="53.34" y1="33.02" x2="53.34" y2="27.94" width="0.1524" layer="91"/>
+<wire x1="55.88" y1="33.02" x2="50.8" y2="33.02" width="0.1524" layer="91"/>
+<wire x1="50.8" y1="33.02" x2="50.8" y2="27.94" width="0.1524" layer="91"/>
 <pinref part="GND2" gate="1" pin="GND"/>
+<pinref part="C3" gate="G$1" pin="2"/>
+<wire x1="50.8" y1="27.94" x2="50.8" y2="22.86" width="0.1524" layer="91"/>
+<wire x1="50.8" y1="35.56" x2="48.26" y2="35.56" width="0.1524" layer="91"/>
+<pinref part="C4" gate="G$1" pin="2"/>
+<wire x1="50.8" y1="27.94" x2="48.26" y2="27.94" width="0.1524" layer="91"/>
+<junction x="50.8" y="35.56"/>
+<junction x="50.8" y="33.02"/>
+<junction x="50.8" y="27.94"/>
+<pinref part="U1" gate="U$1" pin="AGND"/>
+<wire x1="55.88" y1="38.1" x2="50.8" y2="38.1" width="0.1524" layer="91"/>
+<wire x1="50.8" y1="38.1" x2="50.8" y2="35.56" width="0.1524" layer="91"/>
 </segment>
 <segment>
@@
 <wire x1="111.76" y1="106.68" x2="109.22" y2="106.68" width="0.1524" layer="91"/>
 <wire x1="109.22" y1="106.68" x2="109.22" y2="111.76" width="0.1524" layer="91"/>
+<junction x="109.22" y="111.76"/>
+<junction x="109.22" y="106.68"/>
+<wire x1="109.22" y1="106.68" x2="109.22" y2="101.6" width="0.1524" layer="91"/>
+<pinref part="MISC" gate="-1" pin="S"/>
+<wire x1="109.22" y1="101.6" x2="111.76" y2="101.6" width="0.1524" layer="91"/>
 </segment>
 </net>
@@
 <segment>
 <pinref part="ISP1" gate="G$1" pin="VCC"/>
-<wire x1="152.4" y1="33.02" x2="162.56" y2="33.02" width="0.1524" layer="91"/>
-<label x="162.56" y="33.02" size="1.778" layer="95" xref="yes"/>
+<wire x1="152.4" y1="33.02" x2="154.94" y2="33.02" width="0.1524" layer="91"/>
+<label x="154.94" y="33.02" size="1.778" layer="95" xref="yes"/>
 </segment>
 <segment>
@@
 <wire x1="50.8" y1="81.28" x2="48.26" y2="81.28" width="0.1524" layer="91"/>
 <label x="48.26" y="81.28" size="1.778" layer="95" rot="R180" xref="yes"/>
+<junction x="50.8" y="81.28"/>
 </segment>
 <segment>
@@
 <wire x1="154.94" y1="106.68" x2="152.4" y2="106.68" width="0.1524" layer="91"/>
 <wire x1="152.4" y1="106.68" x2="152.4" y2="111.76" width="0.1524" layer="91"/>
+<junction x="152.4" y="111.76"/>
+</segment>
+<segment>
+<pinref part="C3" gate="G$1" pin="1"/>
+<wire x1="40.64" y1="35.56" x2="35.56" y2="35.56" width="0.1524" layer="91"/>
+<label x="35.56" y="35.56" size="1.778" layer="95" rot="R180" xref="yes"/>
 </segment>
 </net>
@@
 <pinref part="U$1" gate="G$1" pin="DI"/>
 <pinref part="ISP1" gate="G$1" pin="MOSI"/>
-<wire x1="152.4" y1="30.48" x2="157.48" y2="30.48" width="0.1524" layer="91"/>
-<wire x1="157.48" y1="30.48" x2="157.48" y2="38.1" width="0.1524" layer="91"/>
-<wire x1="157.48" y1="38.1" x2="127" y2="38.1" width="0.1524" layer="91"/>
+<wire x1="152.4" y1="30.48" x2="165.1" y2="30.48" width="0.1524" layer="91"/>
+<wire x1="165.1" y1="30.48" x2="165.1" y2="38.1" width="0.1524" layer="91"/>
+<wire x1="165.1" y1="38.1" x2="127" y2="38.1" width="0.1524" layer="91"/>
 <wire x1="127" y1="38.1" x2="127" y2="35.56" width="0.1524" layer="91"/>
 <pinref part="U1" gate="U$1" pin="PB3(MOSI/OC2)"/>
@@
 <wire x1="190.5" y1="106.68" x2="187.96" y2="106.68" width="0.1524" layer="91"/>
 <wire x1="187.96" y1="106.68" x2="187.96" y2="111.76" width="0.1524" layer="91"/>
-</segment>
-</net>
+<junction x="187.96" y="111.76"/>
+</segment>
+<segment>
+<pinref part="C4" gate="G$1" pin="1"/>
+<wire x1="40.64" y1="27.94" x2="35.56" y2="27.94" width="0.1524" layer="91"/>
+<label x="35.56" y="27.94" size="1.778" layer="95" rot="R180" xref="yes"/>
+</segment>
+</net>

Commit message: Completed v0.1 of PCB
Signed-off-by: Garrett Greenwood <garrettagreenwood@gmail.com>
Connections:
- net N$10 renamed Z1
- net N$11 renamed X2
- net N$12 renamed Y2
- net N$13 renamed Z3
- net N$14 renamed D_LEFT
- net N$15 renamed D_DOWN
- net N$16 renamed D_RIGHT
- net N$17 renamed D_UP
- net N$18 renamed GCN_SIG
- net N$19 renamed XBOX_RESET
- net N$20 renamed USB_D-
- net N$21 renamed VIEW
- net N$22 renamed XBOX
- net N$23 renamed MENU
- net N$24 renamed R
- net N$25 renamed L
- net N$3 renamed X1
- net N$5 renamed A
- net N$6 renamed B
- net N$7 renamed X
- net N$8 renamed Y
- net N$9 renamed Y1
Changed lines of the file:
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@@
 </segment>
 </net>
-<net name="N$3" class="0">
+<net name="X1" class="0">
 <segment>
 <pinref part="ANALOG" gate="-1" pin="S"/>
@@
 </segment>
 </net>
-<net name="N$9" class="0">
+<net name="Y1" class="0">
 <segment>
 <pinref part="ANALOG" gate="-2" pin="S"/>
@@
 </segment>
 </net>
-<net name="N$10" class="0">
+<net name="Z1" class="0">
 <segment>
 <pinref part="ANALOG" gate="-3" pin="S"/>
@@
 </segment>
 </net>
-<net name="N$11" class="0">
+<net name="X2" class="0">
 <segment>
 <pinref part="ANALOG" gate="-4" pin="S"/>
@@
 </segment>
 </net>
-<net name="N$12" class="0">
+<net name="Y2" class="0">
 <segment>
 <pinref part="U$1" gate="G$1" pin="AO5"/>
@@
 </segment>
 </net>
-<net name="N$13" class="0">
+<net name="Z3" class="0">
 <segment>
 <pinref part="ANALOG" gate="-6" pin="S"/>
@@
 </segment>
 </net>
-<net name="N$14" class="0">
+<net name="D_LEFT" class="0">
 <segment>
 <pinref part="U1" gate="U$1" pin="PB1(OC1A)"/>
@@
 </segment>
 </net>
-<net name="N$15" class="0">
+<net name="D_DOWN" class="0">
 <segment>
 <pinref part="U1" gate="U$1" pin="PB0(ICP)"/>
@@
 </segment>
 </net>
-<net name="N$16" class="0">
+<net name="D_RIGHT" class="0">
 <segment>
 <pinref part="U1" gate="U$1" pin="PD7(AIN1)"/>
@@
 </segment>
 </net>
-<net name="N$17" class="0">
+<net name="D_UP" class="0">
 <segment>
 <pinref part="U1" gate="U$1" pin="PD6(AIN0)"/>
@@
 </segment>
 </net>
-<net name="N$18" class="0">
+<net name="GCN_SIG" class="0">
 <segment>
 <pinref part="U1" gate="U$1" pin="PD5(T1)"/>
@@
 </segment>
 </net>
-<net name="N$19" class="0">
+<net name="XBOX_RESET" class="0">
 <segment>
 <pinref part="U1" gate="U$1" pin="PD4(XCK/T0)"/>
@@
 </segment>
 </net>
-<net name="N$20" class="0">
+<net name="USB_D-" class="0">
 <segment>
 <pinref part="U1" gate="U$1" pin="PD3(INT1)"/>
@@
 </segment>
 </net>
-<net name="N$21" class="0">
+<net name="VIEW" class="0">
 <segment>
 <pinref part="U1" gate="U$1" pin="PD2(INT0)"/>
@@
 </segment>
 </net>
-<net name="N$22" class="0">
+<net name="XBOX" class="0">
 <segment>
 <pinref part="U1" gate="U$1" pin="PD1(TXD)"/>
@@
 </segment>
 </net>
-<net name="N$23" class="0">
+<net name="MENU" class="0">
 <segment>
 <pinref part="U1" gate="U$1" pin="PD0(RXD)"/>
@@
 </segment>
 </net>
-<net name="N$24" class="0">
+<net name="R" class="0">
 <segment>
 <pinref part="U1" gate="U$1" pin="PC5(ADC5/SCL)"/>
@@
 </segment>
 </net>
-<net name="N$25" class="0">
+<net name="L" class="0">
 <segment>
 <pinref part="U1" gate="U$1" pin="PC4(ADC4/SDA)"/>
@@
 </segment>
 </net>
-<net name="N$5" class="0">
+<net name="A" class="0">
 <segment>
 <pinref part="U1" gate="U$1" pin="PC0(ADC0)"/>
@@
 </segment>
 </net>
-<net name="N$6" class="0">
+<net name="B" class="0">
 <segment>
 <pinref part="U1" gate="U$1" pin="PC1(ADC1)"/>
@@
 </segment>
 </net>
-<net name="N$7" class="0">
+<net name="X" class="0">
 <segment>
 <pinref part="U1" gate="U$1" pin="PC2(ADC2)"/>
@@
 </segment>
 </net>
-<net name="N$8" class="0">
+<net name="Y" class="0">
 <segment>
 <pinref part="U1" gate="U$1" pin="PC3(ADC3)"/>

Commit message: Ready to order v0.2 boards
Signed-off-by: Garrett Greenwood <garrettagreenwood@gmail.com>
Parts:
- removed DIGITAL: 53047-09, con-molex:53047-09
- removed Q1: 12MHz, crystal:CRYSTALCTS406
- added Q2: 12MHz, crystal:CRYSTALHC49S
- added R1: 10k, resistor:R-US_R0603
- added U$6: 1X9, headers(2mm):1X9
- ANALOG: value 53047-06 -> 1X6; device con-molex:53047-06 -> headers(2mm):1X6
- DPAD: value 53047-05 -> 1X4; device con-molex:53047-05 -> headers(2mm):1X4
- GCN: value 53047-04 -> 1X4; device con-molex:53047-04 -> headers(2mm):1X4
- MISC: value 53047-05 -> 1X5; device con-molex:53047-05 -> headers(2mm):1X5
- renumbered U$1 to DAC
Connections:
- removed net D_DOWN: DPAD-4.S, U1.PB0(ICP)
- removed net D_LEFT: DPAD-5.S, U1.PB1(OC1A)
- removed net D_RIGHT: DPAD-3.S, U1.PD7(AIN1)
- removed net D_UP: DPAD-2.S, U1.PD6(AIN0)
- removed net USB_D-: MISC-2.S, U1.PD3(INT1)
- removed net XBOX_RESET: MISC-3.S, U1.PD4(XCK/T0)
- new net DPAD-D: DPAD.3, U1.PB0(ICP)
- new net DPAD-L: DPAD.4, U1.PB1(OC1A)
- new net DPAD-R: DPAD.2, U1.PD7(AIN1)
- new net DPAD-U: DPAD.1, U1.PD6(AIN0)
- new net MISC-D-: MISC.4, U1.PD3(INT1)
- new net MISC-RST: MISC.3, U1.PD4(XCK/T0)
- net 3V3: now also GCN.3, MISC.2, R1.2; no longer GCN-3.S, MISC-4.S
- net 5V: now also GCN.4, MISC.1; no longer GCN-4.S, MISC-5.S
- net A: now also U$6.9; no longer DIGITAL-1.S
- net B: now also U$6.8; no longer DIGITAL-2.S
- net GCN_SIG: now also GCN.2, R1.1; no longer GCN-2.S
- net GND: now also GCN.1, MISC.5; no longer DPAD-1.S, GCN-1.S, MISC-1.S
- net L: now also U$6.5; no longer DIGITAL-5.S
- net MENU: now also U$6.3; no longer DIGITAL-7.S
- net N$1: now also Q2.2; no longer Q1.2
- net N$2: now also Q2.1; no longer Q1.1
- net R: now also U$6.4; no longer DIGITAL-6.S
- net VIEW: now also U$6.1; no longer DIGITAL-9.S
- net X: now also U$6.7; no longer DIGITAL-3.S
- net X1: now also ANALOG.1; no longer ANALOG-1.S
- net X2: now also ANALOG.4; no longer ANALOG-4.S
- net XBOX: now also U$6.2; no longer DIGITAL-8.S
- net Y: now also U$6.6; no longer DIGITAL-4.S
- net Y1: now also ANALOG.2; no longer ANALOG-2.S
- net Y2: now also ANALOG.5; no longer ANALOG-5.S
- net Z1: now also ANALOG.3; no longer ANALOG-3.S
- net Z3: now also ANALOG.6; no longer ANALOG-6.S
